Commit message: finishes rosi urdf v1.0

File: urdf/rosi.urdf (robot description, URDF)
Before this commit: robot rosi, 9 links, 8 joints
Links:
- link arm_1: geometry visual mesh filename=package://rosi_defy/urdf/meshes/arm.stl
- link arm_2: geometry visual mesh filename=package://rosi_defy/urdf/meshes/arm.stl
- link arm_3: geometry visual mesh filename=package://rosi_defy/urdf/meshes/arm.stl
- link arm_4: geometry visual mesh filename=package://rosi_defy/urdf/meshes/arm.stl
- link base_link: geometry visual mesh filename=package://rosi_defy/urdf/meshes/rosi_base.stl
- link wheel_1: geometry visual mesh filename=package://rosi_defy/urdf/meshes/wheel.stl
- link wheel_2: geometry visual mesh filename=package://rosi_defy/urdf/meshes/wheel.stl
- link wheel_3: geometry visual mesh filename=package://rosi_defy/urdf/meshes/wheel.stl
- link wheel_4: geometry visual mesh filename=package://rosi_defy/urdf/meshes/wheel.stl

Commit message: fixed rosi arm and wheel joints correctly

File: urdf/rosi.urdf (robot description, URDF)
Before this commit: robot rosi, 9 links, 8 joints
Joints:
- joint joint_wheel_3: origin xyz=0.3152 0.2880 -0.0993 rpy=-1.57 0 3.14 -> xyz=0.3152 0.2880 -0.0993 rpy=-1.57 3.14 0
- joint joint_wheel_4: origin xyz=-0.3152 0.2880 -0.0993 rpy=-1.57 0 3.14 -> xyz=-0.3152 0.2880 -0.0993 rpy=-1.57 3.14 0

Commit message: added velodyne and kinect to the urdf

File: urdf/rosi.urdf (robot description, URDF)
Before this commit: robot rosi, 9 links, 8 joints
Links:
- added link kinect; visual mesh filename=package://rosi_defy/urdf/meshes/kinect.stl
- added link velodyne; visual mesh filename=package://rosi_defy/urdf/meshes/velodyne.stl
Joints:
- added joint joint_kinect: type revolute, parent base_link, child kinect, origin xyz=0.3 0 0.009 rpy=1.57 1.57 0, axis 0 0 1, limit lower=-0.79 upper=0.79 effort=30 velocity=0.79
- added joint joint_velodyne: type fixed, parent base_link, child velodyne, origin xyz=0.242 0.002 0.1655 rpy=0 0.26 0

Commit message: finished ROSI URDF V1

File: urdf/rosi.urdf (robot description, URDF)
Before this commit: robot rosi, 11 links, 10 joints
Links:
- removed link arm_1
- removed link arm_2
- removed link arm_3
- removed link arm_4
- removed link wheel_1
- removed link wheel_2
- removed link wheel_3
- removed link wheel_4
- added link tool_pointer; visual mesh filename=${mesh_folder}/tool_pointer.stl
- link base_link: geometry visual mesh filename=${mesh_folder}/rosi_base.stl
- link kinect: geometry visual mesh filename=${mesh_folder}/kinect.stl
- link velodyne: geometry visual mesh filename=${mesh_folder}/velodyne.stl
Joints:
- removed joint joint_arm_1
- removed joint joint_arm_2
- removed joint joint_arm_3
- removed joint joint_arm_4
- removed joint joint_wheel_1
- removed joint joint_wheel_2
- removed joint joint_wheel_3
- removed joint joint_wheel_4
- added joint joint_l7_tool: type fixed, parent ur5_link_7, child tool_pointer, origin xyz=-0.018 0.034 0.195  rpy=0 0 3.14
- added joint joint_ur5_j1: type revolute, parent base_link, child ur5_link_2, origin xyz=-0.138 -0.067 0.184 rpy=0 0 -1.57, axis 0 0 1
